File: _autosave-RCS_Hardware.kicad_sch (KiCad schematic)
At the start: 28 parts, among them J1 SWD, U1 STM32F401CCU6, U2 AMS1117-3.3, Y1 16MHz

Commit message: added missing USBC foorprint, symbol, and model fixed minor schematic erros setup basic layout for stm32 and capacitors
Parts:
- J1: footprint (none) -> Connector_PinHeader_2.54mm:PinHeader_1x04_P2.54mm_Vertical
- J2: renamed from J?; footprint HRO_TYPE-C-31-M-12 -> USBC:HRO_TYPE-C-31-M-12
- gave numbers to parts that had none: 4
Connections:
- net OSC_IN: now reaches C2.1, U1.5 (PH0), Y1.1
- net OSC_OUT: now reaches C3.1, U1.6 (PH1), Y1.3
- net RADIO_CS: no longer names the net of U1.25 (PB12)
- net SPI2_MISO: no longer names the net of U1.27 (PB14)
- net SPI2_SCK: no longer names the net of U1.26 (PB13)
- net SPI_MOSI: no longer names the net of U1.28 (PB15)
- no-connect marks 22 -> 37
Other:
- note added: "Flash"
- note removed: "M3"
- moved on the sheet: H1, H2, H3, H4, J1
